Commit message: enable rviz2

File: ros2_control_demo_description/diffbot_description/urdf/diffbot_amr1.urdf.xacro (robot description, xacro)
@@ -23,5 +23,5 @@
     </collision>
 		<visual>
-      <origin xyz="1.0 1.0 0" rpy="0 0 0"/>
+      <origin xyz="0 0 0" rpy="0 0 0"/>
       <geometry>
         <box size="${base_width} ${base_length} ${base_height}"/>
@@ -54,5 +54,5 @@
       </collision>
       <visual>
-        <origin xyz="1 1 0" rpy="${PI/2} 0 0"/>
+        <origin xyz="0 0 0" rpy="${PI/2} 0 0"/>
         <geometry>
           <cylinder length="${wheel_len}" radius="${wheel_radius}"/>
@@ -85,5 +85,5 @@
       </collision>
       <visual>
-        <origin xyz="1 1 0" rpy="${PI/2} 0 0"/>
+        <origin xyz="0 0 0" rpy="${PI/2} 0 0"/>
         <geometry>
           <cylinder length="${wheel_len}" radius="${wheel_radius}"/>
@@ -114,5 +114,5 @@
       </collision>
       <visual>
-        <origin xyz="1 1 0" rpy="0 0 0"/>
+        <origin xyz="0 0 0" rpy="0 0 0"/>
         <geometry>
           <sphere radius="${caster_wheel_radius}"/>
@@ -143,5 +143,5 @@
       </collision>
       <visual>
-        <origin xyz="1 1 0" rpy="0 0 0"/>
+        <origin xyz="0 0 0" rpy="0 0 0"/>
         <geometry>
           <sphere radius="${caster_wheel_radius}"/>

File: ros2_control_demo_description/diffbot_description/urdf/diffbot_amr2.urdf.xacro (robot description, xacro)
@@ -10,5 +10,5 @@
   <xacro:property name="wheel_mass" value="0.3" /> <!-- arbitrary value for wheel mass -->
   <xacro:property name="wheel_len" value="0.020" />
-  <xacro:property name="wheel_radius" value="0.015" />
+  <xacro:property name="wheel_radius" value="0.005" />
   <xacro:property name="caster_wheel_mass" value="0.1" /> <!-- arbitrary value for caster wheel mass -->
   <xacro:property name="caster_wheel_radius" value="0.015" />
@@ -22,10 +22,10 @@
       </geometry>
     </collision>
-    <visual>
-      <origin xyz="0 0 0" rpy="0 0 0"/>
+		<visual>
+      <origin xyz="1.0 1.0 0" rpy="0 0 0"/>
       <geometry>
         <box size="${base_width} ${base_length} ${base_height}"/>
       </geometry>
-      <material name="orange"/>
+      <material name="red"/>
     </visual>
     <inertial>
@@ -54,5 +54,5 @@
       </collision>
       <visual>
-        <origin xyz="0 0 0" rpy="${PI/2} 0 0"/>
+        <origin xyz="1 1 0" rpy="${PI/2} 0 0"/>
         <geometry>
           <cylinder length="${wheel_len}" radius="${wheel_radius}"/>
@@ -85,5 +85,5 @@
       </collision>
       <visual>
-        <origin xyz="0 0 0" rpy="${PI/2} 0 0"/>
+        <origin xyz="1 1 0" rpy="${PI/2} 0 0"/>
         <geometry>
           <cylinder length="${wheel_len}" radius="${wheel_radius}"/>
@@ -114,5 +114,5 @@
       </collision>
       <visual>
-        <origin xyz="0 0 0" rpy="0 0 0"/>
+        <origin xyz="1 1 0" rpy="0 0 0"/>
         <geometry>
           <sphere radius="${caster_wheel_radius}"/>
@@ -143,5 +143,5 @@
       </collision>
       <visual>
-        <origin xyz="0 0 0" rpy="0 0 0"/>
+        <origin xyz="1 1 0" rpy="0 0 0"/>
         <geometry>
           <sphere radius="${caster_wheel_radius}"/>

File: ros2_control_demo_description/diffbot_description/urdf/diffbot_system_amr1.urdf.xacro (robot description, xacro)
@@ -11,5 +11,5 @@
   <xacro:arg name="fake_sensor_commands" default="false" />
   <xacro:arg name="prefix" default="" />
-  <xacro:include filename="$(find diffbot_description)/urdf/diffbot1.urdf.xacro" />
+  <xacro:include filename="$(find diffbot_description)/urdf/diffbot_amr1.urdf.xacro" />
   <!-- Import all Gazebo-customization elements, including Gazebo colors -->
   <xacro:include filename="$(find diffbot_description)/gazebo/diffbot.gazebo.xacro" />
@@ -17,5 +17,5 @@
   <xacro:include filename="$(find diffbot_description)/gazebo/diffbot.materials.xacro" />
   <!-- Import diffbot ros2_control description -->
-  <xacro:include filename="$(find diffbot_description)/ros2_control/diffbot_system.ros2_control.xacro" />
+  <xacro:include filename="$(find diffbot_description)/ros2_control/diffbot_system_amr1.ros2_control.xacro" />
   <xacro:diffbot prefix="$(arg prefix)" />
   <xacro:diffbot_gazebo prefix="$(arg prefix)" />

File: ros2_control_demo_description/diffbot_description/urdf/diffbot_system_amr2.urdf.xacro (robot description, xacro)
@@ -11,5 +11,5 @@
   <xacro:arg name="fake_sensor_commands" default="false" />
   <xacro:arg name="prefix" default="" />
-  <xacro:include filename="$(find diffbot_description)/urdf/diffbot.urdf.xacro" />
+  <xacro:include filename="$(find diffbot_description)/urdf/diffbot_amr2.urdf.xacro" />
   <!-- Import all Gazebo-customization elements, including Gazebo colors -->
   <xacro:include filename="$(find diffbot_description)/gazebo/diffbot.gazebo.xacro" />
@@ -17,5 +17,5 @@
   <xacro:include filename="$(find diffbot_description)/gazebo/diffbot.materials.xacro" />
   <!-- Import diffbot ros2_control description -->
-  <xacro:include filename="$(find diffbot_description)/ros2_control/diffbot_system.ros2_control.xacro" />
+  <xacro:include filename="$(find diffbot_description)/ros2_control/diffbot_system_amr2.ros2_control.xacro" />
   <xacro:diffbot prefix="$(arg prefix)" />
   <xacro:diffbot_gazebo prefix="$(arg prefix)" />
